Commit message: 改外参

File: workspace_auv/src/auv_description/urdf/auv.urdf (robot description, URDF)
Before this commit: robot youlong_auv, 15 links, 14 joints
Joints:
- joint disc_claw_mount: origin xyz=-0.400 0 0.290 rpy=3.141592653589793 -1.5707963267948966 0 -> xyz=-0.300 0 0.290 rpy=3.141592653589793 -1.5707963267948966 0
- joint hairpin_claw_mount: origin xyz=0.280 0 0.130 rpy=3.141592653589793 -1.5707963267948966 0 -> xyz=0.320 0 0.130 rpy=3.141592653589793 -1.5707963267948966 0

Commit message: 最后一舞agx代码

File: workspace_auv/src/auv_description/urdf/auv.urdf (robot description, URDF)
Before this commit: robot youlong_auv, 15 links, 14 joints
Joints:
- joint disc_claw_mount: origin xyz=-0.35 0 0.290 rpy=3.141592653589793 -1.5707963267948966 0 -> xyz=-0.32 0 0.290 rpy=3.141592653589793 -1.5707963267948966 0
- joint hairpin_claw_mount: origin xyz=0.350 0 0.130 rpy=3.141592653589793 -1.5707963267948966 0 -> xyz=0.335 0 0.130 rpy=3.141592653589793 -1.5707963267948966 0
