Commit message: 增加rviz

File: workspace_auv/src/auv_description/urdf/auv.urdf (robot description, URDF)
Before this commit: robot youlong_auv, 13 links, 12 joints
Links:
- link base_link: geometry visual mesh filename=package://uv_rviz/meshes/youlong/battery_pod.obj scale=0.001 0.001 0.001; visual mesh filename=package://uv_rviz/meshes/youlong/propeller.obj scale=0.35 0.35 0.35
- link downward_camera_link: geometry visual box size=0.075 0.14 0.045
- link downward_left_camera_optical_frame: geometry visual cylinder length=0.012 radius=0.013
- link downward_right_camera_optical_frame: geometry visual cylinder length=0.012 radius=0.013
- link front_camera_link: geometry visual box size=0.09 0.14 0.055
- link front_left_camera_optical_frame: geometry visual cylinder length=0.014 radius=0.014
- link front_right_camera_optical_frame: geometry visual cylinder length=0.014 radius=0.014
- link imu_link: geometry visual box size=0.075 0.075 0.04
- link usbl_array_geometry_center: geometry visual sphere 
- link usbl_link: geometry visual cylinder length=0.025 radius=0.042
- link usbl_transducer_a1: geometry visual cylinder length=0.012 radius=0.012
- link usbl_transducer_a2: geometry visual cylinder length=0.012 radius=0.012
- link usbl_transducer_a3: geometry visual cylinder length=0.012 radius=0.012

File: workspace_sim/src/uv_sim_description/urdf/auv_sim.urdf (robot description, URDF)
Before this commit: robot youlong_auv, 10 links, 9 joints
Links:
- link base_link: geometry visual mesh filename=package://uv_rviz/meshes/youlong/battery_pod.obj scale=0.001 0.001 0.001; visual mesh filename=package://uv_rviz/meshes/youlong/propeller.obj scale=0.35 0.35 0.35
- link downward_camera_link: geometry visual box size=0.075 0.14 0.045
- link downward_left_camera_optical_frame: geometry visual cylinder length=0.012 radius=0.013
- link downward_right_camera_optical_frame: geometry visual cylinder length=0.012 radius=0.013
- link dvl_link: geometry visual cylinder length=0.07 radius=0.045
- link front_camera_link: geometry visual box size=0.09 0.14 0.055
- link front_left_camera_optical_frame: geometry visual cylinder length=0.014 radius=0.014
- link front_right_camera_optical_frame: geometry visual cylinder length=0.014 radius=0.014
- link imu_link: geometry visual box size=0.075 0.075 0.04
- link usbl_link: geometry visual cylinder length=0.025 radius=0.042

Commit message: 修改摄像头映射,同时反转前视

File: workspace_auv/src/auv_description/urdf/auv.urdf (robot description, URDF)
Before this commit: robot youlong_auv, 13 links, 12 joints
Joints:
- joint front_left_camera_mount: origin xyz=0 -0.05 0 rpy=1.5708 0 1.5708 -> xyz=0 -0.05 0 rpy=-1.5708 0 -1.5708
- joint front_right_camera_mount: origin xyz=0 0.05 0 rpy=1.5708 0 1.5708 -> xyz=0 0.05 0 rpy=-1.5708 0 -1.5708

Commit message: 改下视方向,launch缩进

File: workspace_auv/src/auv_description/urdf/auv.urdf (robot description, URDF)
Before this commit: robot youlong_auv, 13 links, 12 joints
Joints:
- joint downward_left_camera_mount: origin xyz=0 -0.05 0 rpy=0 0 1.5708 -> xyz=0 -0.05 0 rpy=0 0 -1.5708
- joint downward_right_camera_mount: origin xyz=0 0.05 0 rpy=0 0 1.5708 -> xyz=0 0.05 0 rpy=0 0 -1.5708

Commit message: 修改launch,增强camera节点启动鲁棒性

File: workspace_auv/src/auv_description/urdf/auv.urdf (robot description, URDF)
Before this commit: robot youlong_auv, 13 links, 12 joints
Joints:
- joint downward_left_camera_mount: origin xyz=0 -0.05 0 rpy=0 0 -1.5708 -> xyz=0 -0.03 0 rpy=0 0 -1.5708
- joint downward_right_camera_mount: origin xyz=0 0.05 0 rpy=0 0 -1.5708 -> xyz=0 0.03 0 rpy=0 0 -1.5708
- joint front_left_camera_mount: origin xyz=0 -0.05 0 rpy=-1.5708 0 -1.5708 -> xyz=0 -0.03 0 rpy=-1.5708 0 -1.5708
- joint front_right_camera_mount: origin xyz=0 0.05 0 rpy=-1.5708 0 -1.5708 -> xyz=0 0.03 0 rpy=-1.5708 0 -1.5708

Commit message: 更正双目外参

File: workspace_auv/src/auv_description/urdf/auv.urdf (robot description, URDF)
Before this commit: robot youlong_auv, 13 links, 12 joints
Joints:
- joint downward_left_camera_mount: origin xyz=0 -0.03 0 rpy=0 0 -1.5708 -> xyz=0 -0.03058633655786893 0 rpy=0 0 -1.5708
- joint downward_right_camera_mount: origin xyz=0 0.03 0 rpy=0 0 -1.5708 -> xyz=0 0.03058633655786893 0 rpy=0 0 -1.5708

Commit message: 修正双目图像顺序与三维 TF，并更新夹爪坐标、任务逻辑和硬件心跳配置

File: workspace_auv/src/auv_description/urdf/auv.urdf (robot description, URDF)
Before this commit: robot youlong_auv, 13 links, 12 joints
Links:
- added link disc_claw_link
- added link hairpin_claw_link
- link usbl_array_geometry_center: geometry visual sphere radius=0.012
Joints:
- added joint disc_claw_mount: type fixed, parent base_link, child disc_claw_link, origin xyz=-0.430 0 0.290 rpy=3.141592653589793 -1.5707963267948966 0
- added joint hairpin_claw_mount: type fixed, parent base_link, child hairpin_claw_link, origin xyz=0.080 0 0.130 rpy=3.141592653589793 -1.5707963267948966 0
- joint downward_left_camera_mount: origin xyz=0 -0.03058633655786893 0 rpy=0 0 -1.5708 -> xyz=0 -0.03058633655786893 0 rpy=0 0 1.5707963267948966
- joint downward_right_camera_mount: origin xyz=0 0.03058633655786893 0 rpy=0 0 -1.5708 -> xyz=0 0.03058633655786893 0 rpy=0 0 1.5707963267948966
- joint front_left_camera_mount: origin xyz=0 -0.03 0 rpy=-1.5708 0 -1.5708 -> xyz=0 -0.03 0 rpy=1.5707963267948966 0 1.5707963267948966
- joint front_right_camera_mount: origin xyz=0 0.03 0 rpy=-1.5708 0 -1.5708 -> xyz=0 0.03 0 rpy=1.5707963267948966 0 1.5707963267948966

Commit message: 设置外参,微调任务参数

File: workspace_auv/src/auv_description/urdf/auv.urdf (robot description, URDF)
Before this commit: robot youlong_auv, 15 links, 14 joints
Joints:
- joint disc_claw_mount: origin xyz=-0.430 0 0.290 rpy=3.141592653589793 -1.5707963267948966 0 -> xyz=-0.320 0 0.290 rpy=3.141592653589793 -1.5707963267948966 0

Commit message: 外参

File: workspace_auv/src/auv_description/urdf/auv.urdf (robot description, URDF)
Before this commit: robot youlong_auv, 15 links, 14 joints
Joints:
- joint disc_claw_mount: origin xyz=-0.320 0 0.290 rpy=3.141592653589793 -1.5707963267948966 0 -> xyz=-0.400 0 0.290 rpy=3.141592653589793 -1.5707963267948966 0
- joint hairpin_claw_mount: origin xyz=0.080 0 0.130 rpy=3.141592653589793 -1.5707963267948966 0 -> xyz=0.280 0 0.130 rpy=3.141592653589793 -1.5707963267948966 0

Commit message: 123

File: workspace_auv/src/auv_description/urdf/auv.urdf (robot description, URDF)
Before this commit: robot youlong_auv, 15 links, 14 joints
Joints:
- joint disc_claw_mount: origin xyz=-0.300 0 0.290 rpy=3.141592653589793 -1.5707963267948966 0 -> xyz=-0.340 0 0.290 rpy=3.141592653589793 -1.5707963267948966 0

Commit message: 任务调整,加细调整

File: workspace_auv/src/auv_description/urdf/auv.urdf (robot description, URDF)
Before this commit: robot youlong_auv, 15 links, 14 joints
Joints:
- joint disc_claw_mount: origin xyz=-0.340 0 0.290 rpy=3.141592653589793 -1.5707963267948966 0 -> xyz=-0.400 0 0.290 rpy=3.141592653589793 -1.5707963267948966 0
- joint hairpin_claw_mount: origin xyz=0.320 0 0.130 rpy=3.141592653589793 -1.5707963267948966 0 -> xyz=0.280 0 0.130 rpy=3.141592653589793 -1.5707963267948966 0

Commit message: 外参

File: workspace_auv/src/auv_description/urdf/auv.urdf (robot description, URDF)
Before this commit: robot youlong_auv, 15 links, 14 joints
Joints:
- joint disc_claw_mount: origin xyz=-0.400 0 0.290 rpy=3.141592653589793 -1.5707963267948966 0 -> xyz=-0.30 0 0.290 rpy=3.141592653589793 -1.5707963267948966 0

Commit message: 下潜代码

File: workspace_auv/src/auv_description/urdf/auv.urdf (robot description, URDF)
Before this commit: robot youlong_auv, 15 links, 14 joints
Joints:
- joint disc_claw_mount: origin xyz=-0.30 0 0.290 rpy=3.141592653589793 -1.5707963267948966 0 -> xyz=-0.25 0 0.290 rpy=3.141592653589793 -1.5707963267948966 0

Commit message: 改过门

File: workspace_auv/src/auv_description/urdf/auv.urdf (robot description, URDF)
Before this commit: robot youlong_auv, 15 links, 14 joints
Joints:
- joint disc_claw_mount: origin xyz=-0.25 0 0.290 rpy=3.141592653589793 -1.5707963267948966 0 -> xyz=-0.20 0 0.290 rpy=3.141592653589793 -1.5707963267948966 0

Commit message: 123

File: workspace_auv/src/auv_description/urdf/auv.urdf (robot description, URDF)
Before this commit: robot youlong_auv, 15 links, 14 joints
Joints:
- joint disc_claw_mount: origin xyz=-0.20 0 0.290 rpy=3.141592653589793 -1.5707963267948966 0 -> xyz=-0.35 0 0.290 rpy=3.141592653589793 -1.5707963267948966 0

Commit message: urdf

File: workspace_auv/src/auv_description/urdf/auv.urdf (robot description, URDF)
Before this commit: robot youlong_auv, 15 links, 14 joints
Joints:
- joint hairpin_claw_mount: origin xyz=0.280 0 0.130 rpy=3.141592653589793 -1.5707963267948966 0 -> xyz=0.230 0 0.130 rpy=3.141592653589793 -1.5707963267948966 0

Commit message: bline

File: workspace_auv/src/auv_description/urdf/auv.urdf (robot description, URDF)
Before this commit: robot youlong_auv, 15 links, 14 joints
Joints:
- joint hairpin_claw_mount: origin xyz=0.230 0 0.130 rpy=3.141592653589793 -1.5707963267948966 0 -> xyz=0.350 0 0.130 rpy=3.141592653589793 -1.5707963267948966 0

Commit message: 123

File: workspace_auv/src/auv_description/urdf/auv.urdf (robot description, URDF)
Before this commit: robot youlong_auv, 15 links, 14 joints
Joints:
- joint disc_claw_mount: origin xyz=-0.35 0 0.290 rpy=3.141592653589793 -1.5707963267948966 0 -> xyz=-0.32 0 0.290 rpy=3.141592653589793 -1.5707963267948966 0
- joint hairpin_claw_mount: origin xyz=0.350 0 0.130 rpy=3.141592653589793 -1.5707963267948966 0 -> xyz=0.310 0 0.130 rpy=3.141592653589793 -1.5707963267948966 0

Commit message: 佛祖保佑二版

File: workspace_auv/src/auv_description/urdf/auv.urdf (robot description, URDF)
Before this commit: robot youlong_auv, 15 links, 14 joints
Joints:
- joint disc_claw_mount: origin xyz=-0.32 0 0.290 rpy=3.141592653589793 -1.5707963267948966 0 -> xyz=-0.28 0 0.290 rpy=3.141592653589793 -1.5707963267948966 0
- joint hairpin_claw_mount: origin xyz=0.335 0 0.130 rpy=3.141592653589793 -1.5707963267948966 0 -> xyz=0.35 0 0.130 rpy=3.141592653589793 -1.5707963267948966 0
